Commit message: Copied robot and simulation files

File: three_pi_description/urdf/sensors_three_pi.xacro (robot description, xacro)
@@ -1,5 +1,5 @@
 <?xml version="1.0" ?>
 <robot name="three_pi_sensors" xmlns:xacro="https://www.ros.org/wiki/xacro">
-    <!-- camera link 1 (original) -->
+    <!-- camera link -->
     <link name="camera_link">
         <collision>
@@ -12,67 +12,9 @@
     <joint name="camera_joint" type="fixed">
         <!-- <origin xyz="0.08 0.0 0.15" rpy="0.0 ${pi/2} 0.0" /> -->
-        <origin xyz="0.08 0.0 0.15" rpy="0.0 ${pi/4} 0.0" />
-        <!-- <origin xyz="0.08 0.0 0.15" rpy="0.0 ${pi/7} 0.0" /> -->
-		<parent link="chassis_link" />
+        <!--<origin xyz="0.08 0.0 0.15" rpy="0.0 ${pi/4} 0.0" /> -->
+        <origin xyz="0.08 0.0 0.15" rpy="0.0 ${pi/7} 0.0" />
+        <parent link="chassis_link" />
         <child link="camera_link" />
     </joint>
-	<!-- camera link 2 (left) -->
-	<link name="camera_link_2">
-	<collision>
-		<origin xyz="0.0 0.0 0.0" rpy="0.0 0.0 0.0" />
-		<geometry>
-			<box size="0.01 0.01 0.01" />
-		</geometry>
-	</collision>
-    </link>
-    <joint name="camera_joint_2" type="fixed">
-        <!-- <origin xyz="0.08 0.0 0.15" rpy="0.0 ${pi/2} 0.0" /> -->
-        <origin xyz="0.08 0.1 0.15" rpy="0.0 ${pi/4} 0.0" />
-        <!-- <origin xyz="0.08 0.0 0.15" rpy="0.0 ${pi/7} 0.0" /> -->
-        <parent link="chassis_link" />
-        <child link="camera_link_2" />
-    </joint>
-	<!-- camera link 3 (right) -->
-	<link name="camera_link_3">
-	<collision>
-		<origin xyz="0.0 0.0 0.0" rpy="0.0 0.0 0.0" />
-		<geometry>
-			<box size="0.01 0.01 0.01" />
-		</geometry>
-	</collision>
-    </link>
-    <joint name="camera_joint_3" type="fixed">
-        <!-- <origin xyz="0.08 0.0 0.15" rpy="0.0 ${pi/2} 0.0" /> -->
-        <origin xyz="0.08 -0.1 0.15" rpy="0.0 ${pi/4} 0.0" />
-        <!-- <origin xyz="0.08 0.0 0.15" rpy="0.0 ${pi/7} 0.0" /> -->
-        <parent link="chassis_link" />
-        <child link="camera_link_3" />
-    </joint>
-	<!-- sonar sensor -->
-	<joint name="sonar_front_joint" type="fixed">
-		<axis xyz="0 1 0" />
-		<origin rpy="0 0 0" xyz="0.5 0 0.25" />
-		<parent link="chassis_link"/>
-		<child link="base_sonar_front"/>
-	</joint>
-	<link name="base_sonar_front">
-		<collision>
-		  <origin xyz="0 0 0" rpy="0 0 0"/>
-		  <geometry>
-			<box size="0.01 0.01 0.01"/>
-		  </geometry>
-		</collision>
-		<visual>
-		  <origin xyz="0 0 0" rpy="0 0 0"/>
-		  <geometry>
-			<box size="0.01 0.01 0.01"/>
-		  </geometry>
-		</visual>
-		<inertial>
-		  <mass value="1e-5" />
-		  <origin xyz="0 0 0" rpy="0 0 0"/>
-		  <inertia ixx="1e-6" ixy="0" ixz="0" iyy="1e-6" iyz="0" izz="1e-6" />
-		</inertial>
-	</link>
     <!-- lidar link -->
     <link name="lidar_link">

File: three_pi_description_copy/urdf/plugins_three_pi_copy.xacro (robot description, xacro)
@@ -4,5 +4,5 @@
     <xacro:arg name="laser_visual" default="false" />
     <xacro:arg name="imu_visual" default="false" />
-    <!-- camera plugin -->
+    <!-- camera plugin 1 (original) -->
     <gazebo reference="camera_link">
         <sensor type="camera" name="3Pi Camera">
@@ -11,18 +11,21 @@
             <camera>
                 <horizontal_fov>1.085595</horizontal_fov>
-                <!--<image>
+                <image>
                     <width>640</width>
                     <height>480</height>
                     <format>R8G8B8</format>
-                </image> -->
-				<image>
+                </image>
+				<!---<image>
                     <width>50</width>
                     <height>1</height>
-                    <format>R8G8B8</format>
-                </image>
+                    <format>L8</format>
+                </image> -->
                 <clip>
                     <near>0.1</near>
                     <far>1.0</far>
                 </clip>
+				<!--<save enabled="true">
+					<path>/home/elisabeth/Dokumente/GazeboImages/v3</path>
+				</save>-->
             </camera>
             <plugin name="camera_controller" filename="libgazebo_ros_camera.so">
@@ -42,4 +45,124 @@
         </sensor>
     </gazebo>
+    <!-- camera plugin 2 (left)-->
+    <gazebo reference="camera_link_2">
+        <sensor type="camera" name="3Pi Camera">
+            <always_on>true</always_on>
+            <visualize>$(arg camera_visual)</visualize>
+            <camera>
+                <horizontal_fov>1.085595</horizontal_fov>
+                <image>
+                    <width>640</width>
+                    <height>480</height>
+                    <format>R8G8B8</format>
+                </image>
+				<!---<image>
+                    <width>50</width>
+                    <height>1</height>
+                    <format>L8</format>
+                </image> -->
+                <clip>
+                    <near>0.1</near>
+                    <far>1.0</far>
+                </clip>
+				<!--<save enabled="true">
+					<path>/home/elisabeth/Dokumente/GazeboImages/v3</path>
+				</save>-->
+            </camera>
+            <plugin name="camera_controller_2" filename="libgazebo_ros_camera.so">
+                <alwaysOn>true</alwaysOn>
+                <updateRate>0.0</updateRate> <!-- 30 -->
+                <cameraName>camera_2</cameraName>
+                <frameName>camera_rgb_optical_frame_2</frameName>
+                <imageTopicName>image_raw_2</imageTopicName>
+                <cameraInfoTopicName>rgb/camera_info_2</cameraInfoTopicName>
+                <hackBaseline>0.07</hackBaseline>
+                <distortionK1>0.0</distortionK1>
+                <distortionK2>0.0</distortionK2>
+                <distortionK3>0.0</distortionK3>
+                <distortionT1>0.0</distortionT1>
+                <distortionT2>0.0</distortionT2>
+            </plugin>
+        </sensor>
+    </gazebo>
+    <!-- camera plugin 3 (right)-->
+    <gazebo reference="camera_link_3">
+        <sensor type="camera" name="3Pi Camera">
+            <always_on>true</always_on>
+            <visualize>$(arg camera_visual)</visualize>
+            <camera>
+                <horizontal_fov>1.085595</horizontal_fov>
+                <image>
+                    <width>640</width>
+                    <height>480</height>
+                    <format>R8G8B8</format>
+                </image>
+				<!---<image>
+                    <width>50</width>
+                    <height>1</height>
+                    <format>L8</format>
+                </image> -->
+                <clip>
+                    <near>0.1</near>
+                    <far>1.0</far>
+                </clip>
+				<!--<save enabled="true">
+					<path>/home/elisabeth/Dokumente/GazeboImages/v3</path>
+				</save>-->
+            </camera>
+            <plugin name="camera_controller_3" filename="libgazebo_ros_camera.so">
+                <alwaysOn>true</alwaysOn>
+                <updateRate>0.0</updateRate> <!-- 30 -->
+                <cameraName>camera_3</cameraName>
+                <frameName>camera_rgb_optical_frame_3</frameName>
+                <imageTopicName>image_raw_3</imageTopicName>
+                <cameraInfoTopicName>rgb/camera_info_3</cameraInfoTopicName>
+                <hackBaseline>0.07</hackBaseline>
+                <distortionK1>0.0</distortionK1>
+                <distortionK2>0.0</distortionK2>
+                <distortionK3>0.0</distortionK3>
+                <distortionT1>0.0</distortionT1>
+                <distortionT2>0.0</distortionT2>
+            </plugin>
+        </sensor>
+    </gazebo>
+	<!-- sonar sensor plugin -->
+	<gazebo reference="base_sonar_front">
+	   <sensor type="ray" name="TeraRanger">
+		  <pose>0 0 0 0 0 0</pose>
+		  <visualize>true</visualize>
+		  <update_rate>50</update_rate>
+		  <ray>
+			 <scan>
+				<horizontal>
+				   <samples>10</samples>
+				   <resolution>1</resolution>
+				   <min_angle>-0.14835</min_angle>
+				   <max_angle>0.14835</max_angle>
+				</horizontal>
+				<vertical>
+				   <samples>10</samples>
+				   <resolution>1</resolution>
+				   <min_angle>-0.14835</min_angle>
+				   <max_angle>0.14835</max_angle>
+				</vertical>
+			 </scan>
+			 <range>
+				<min>0.01</min>
+				<max>10</max>
+				<resolution>0.02</resolution>
+			 </range>
+		  </ray>
+		  <plugin filename="libgazebo_ros_range.so" name="gazebo_ros_range">
+			 <gaussianNoise>0.005</gaussianNoise>
+			 <alwaysOn>true</alwaysOn>
+			 <updateRate>30</updateRate>
+			 <topicName>sensor/sonar_front</topicName>
+			 <frameName>base_sonar_front</frameName>
+			 <radiation>ultrasound</radiation>
+			 <fov>0.2967</fov>
+		  </plugin>
+	   </sensor>
+   </gazebo>
     <!-- lidar plugin -->
     <gazebo reference="lidar_link">
