Commit message: Added distance measurement node and obstacles

File: three_pi_description_copy/urdf/plugins_three_pi_copy.xacro (robot description, xacro)
@@ -142,13 +142,13 @@
 				</horizontal>
 				<vertical>
-				   <samples>10</samples>
+				   <samples>1</samples>
 				   <resolution>1</resolution>
-				   <min_angle>-0.14835</min_angle>
-				   <max_angle>0.14835</max_angle>
+				   <min_angle>-0.04835</min_angle>
+				   <max_angle>0.04835</max_angle>
 				</vertical>
 			 </scan>
 			 <range>
 				<min>0.01</min>
-				<max>10</max>
+				<max>1</max>
 				<resolution>0.02</resolution>
 			 </range>

File: three_pi_description_copy/urdf/sensors_three_pi_copy.xacro (robot description, xacro)
@@ -52,24 +52,18 @@
 	<joint name="sonar_front_joint" type="fixed">
 		<axis xyz="0 1 0" />
-		<origin rpy="0 0 0" xyz="0.5 0 0.25" />
+		<origin rpy="0 -0.15 0" xyz="0.05 0 0.085" />
 		<parent link="chassis_link"/>
 		<child link="base_sonar_front"/>
 	</joint>
 	<link name="base_sonar_front">
-		<collision>
-		  <origin xyz="0 0 0" rpy="0 0 0"/>
+		<visual>
+		  <origin xyz="0.0 0.0 0.0" rpy="0.0 0.0 0.0"/>
 		  <geometry>
-			<box size="0.01 0.01 0.01"/>
-		  </geometry>
-		</collision>
-		<visual>
-		  <origin xyz="0 0 0" rpy="0 0 0"/>
-		  <geometry>
-			<box size="0.01 0.01 0.01"/>
+			<box size="0.05 0.05 0.05"/>
 		  </geometry>
 		</visual>
 		<inertial>
 		  <mass value="1e-5" />
-		  <origin xyz="0 0 0" rpy="0 0 0"/>
+		  <origin xyz="0.0 0.0 0.0" rpy="0.0 0.0 0.0"/>
 		  <inertia ixx="1e-6" ixy="0" ixz="0" iyy="1e-6" iyz="0" izz="1e-6" />
 		</inertial>
